File: display-esp32-addon_1.kicad_pcb (KiCad board)
At the start: 2 copper layers, 100 x 50 mm, 6 parts, among them J1 Conn_01x07_Socket, J2 Conn_01x07_Socket

Commit message: agregando fiducials
Parts:
- added FID1: Fiducial, Fiducial:Fiducial_1mm_Mask2mm, F.Cu at (109.9, 73.7)
- added FID2: Fiducial, Fiducial:Fiducial_1mm_Mask2mm, F.Cu at (192.4, 118.2)
- added FID3: Fiducial, Fiducial:Fiducial_1mm_Mask2mm, F.Cu at (192.4, 73.7)
- added FID4: Fiducial, Fiducial:Fiducial_1mm_Mask2mm, B.Cu at (109.9, 118.2)
- added FID5: Fiducial, Fiducial:Fiducial_1mm_Mask2mm, B.Cu at (109.9, 73.7)
- added FID6: Fiducial, Fiducial:Fiducial_1mm_Mask2mm, B.Cu at (192.4, 118.2)
- added FID7: Fiducial, Fiducial:Fiducial_1mm_Mask2mm, F.Cu at (109.9, 118.2)
- added FID8: Fiducial, Fiducial:Fiducial_1mm_Mask2mm, B.Cu at (192.4, 73.7)
